File: hardware/stick.kicad_pcb (KiCad board)
At the start: 4 copper layers, 46.5 x 17.4 mm, 11 parts, among them J1 USB-A edge plug, U1 ESP32-S3-MINI-1-N4, U2 AP2112K-3.3

Commit message: Rebuild site in plain JS: home presentation, explorer with Guide and Files tabs, single-stick logo, PCB fixes
Co-Authored-By: Claude Sonnet 5.5 <noreply@anthropic.com>
Parts:
- added C3: 100nF, C_0402_1005Metric, B.Cu at (8.62, 14.6)
Other:
- board text added: "D1"
- board text added: "v1"
